File: Alu.kicad_sch (KiCad schematic)
At the start: 9 parts, among them U20 74LS153, U21 74LS153, U22 Am2903, U23 Am2903, U24 Am2903, U25 Am2903, U26 Am2918, U27 Am2922, U28 Am2922

Commit message: More parts of the schema
Parts:
- removed U23, U24, U25: Am2903, Package_DIP:DIP-48_W15.24mm, symbol frits:am2903
- added R2: 1K, symbol Device:R
- added U20, U21: Am2920, Package_DIP:DIP-22_W10.16mm, symbol frits:Am2920
- added U27, U28, U29: Am2903, Package_DIP:DIP-48_W15.24mm, symbol frits:am2903
- added U30: Am2902A, Package_DIP:DIP-16_W10.16mm, symbol frits:Am2902
- added U34, U35, U36: Am2922, Package_DIP:DIP-20_W7.62mm, symbol frits:Am2922
- added U38: 74LS157, symbol 74xx:74LS157
- renumbered U20 to U22, U21 to U23, U26 to U24, U27 to U25, U22 to U26, U28 to U33
Connections:
- net +5V: now also U26.36 (Vcc), U26.39 (~{LSS}), U33. (Vcc), R2.1, U20.1 (~{CLR}), U20.22 (Vcc), U21.1 (~{CLR}), U21.22 (Vcc), U27.36 (Vcc), U28.36 (Vcc), U29.36 (Vcc), U30.16 (Vcc), U34. (Vcc), U35. (Vcc), U36. (Vcc), U38.16 (VCC)
- net GND: now also U26.13 (GND), U26.15 (~{OEY}), U26.40 (~{MSS/WRITE}), U33. (Vcc), U20.11 (GND), U21.11 (GND), U27.13 (GND), U27.15 (~{OEY}), U27.39 (~{LSS}), U27.40 (~{MSS/WRITE}), U28.13 (GND), U28.15 (~{OEY}), U28.39 (~{LSS}), U28.40 (~{MSS/WRITE}), U29.13 (GND), U29.15 (~{OEY}), U29.39 (~{LSS}), U30.8 (GND), U34. (Vcc), U35. (Vcc), U36. (Vcc), U38.15 (E), U38.8 (GND)
- net clock: now also U26.43 (CP), U33. (Vcc), U20.10 (CLK), U21.10 (CLK), U27.43 (CP), U28.43 (CP), U29.43 (CP), U34. (Vcc), U35. (Vcc), U36. (Vcc)
- net cy: now also U26.11 (Cn+4)
- net n: now also U26. (SIGN)
- net ovf: now also U26.12 (~{P}/OVR)
- net at U26.1 (QIO0): now also U27.48 (QIO3)
- net at U26.10 (CN): now also U30.9 (Cn+Z)
- net Y12: now reaches U26.16 (Y0)
- net Y13: now reaches U26.17 (Y1)
- net Y14: now reaches U26.18 (Y2)
- net Y15: now reaches U26.19 (Y3)
- net pl10: now reaches U26.2 (~{EA})
- net pl10: now also U27.2 (~{EA}), U28.2 (~{EA}), U29.2 (~{EA})
- net at U26.20 (SIO0): now also U27.21 (SIO3)
- net SH: now reaches U26.21 (SIO3)
- net SH: now also U23.5 (I1a), U34. (Vcc), U35. (Vcc), U36. (Vcc)
- net at U26.22 (Z): now also R2.2, U27.22 (Z), U28.22 (Z), U29.22 (Z)
- net DB12: now reaches U26.23 (DB0)
- net DB12: now also U20.12 (Y4), U27.23 (DB0), U28.23 (DB0), U29.23 (DB0)
- net DB13: now reaches U26.24 (DB1)
- net DB13: now also U20.15 (Y5), U27.24 (DB1), U28.24 (DB1), U29.24 (DB1)
- net DB14: now reaches U26.25 (DB2)
- net DB14: now also U20.16 (Y6), U27.25 (DB2), U28.25 (DB2), U29.25 (DB2)
- net DB15: now reaches U26.26 (DB3)
- net DB15: now also U20.19 (Y7), U27.26 (DB3), U28.26 (DB3), U29.26 (DB3)
- net alu_a3: now reaches U26.27 (A3)
- net alu_a3: now also U27.27 (A3), U28.27 (A3), U29.27 (A3)
- net alu_a2: now reaches U26.28 (A2)
- net alu_a2: now also U27.28 (A2), U28.28 (A2), U29.28 (A2)
- net alu_a1: now reaches U26.29 (A1)
- net alu_a1: now also U27.29 (A1), U28.29 (A1), U29.29 (A1)
- net DA12: now reaches U26.3 (DA0)
- net DA12: now also U27.3 (DA0), U28.3 (DA0), U29.3 (DA0)
- net alu_a0: now reaches U26.30 (A0)
- net alu_a0: now also U27.30 (A0), U28.30 (A0), U29.30 (A0)
- net pl11: now reaches U26.31 (~{OEB})
- net pl11: now also U27.31 (~{OEB}), U28.31 (~{OEB}), U29.31 (~{OEB})
- net pl8: now reaches U26.32 (I8)
- net pl8: now also U33. (Vcc), U27.32 (I8), U28.32 (I8), U29.32 (I8), U34. (Vcc)
- net pl7: now reaches U26.33 (I7)
- net pl7: now also U27.33 (I7), U28.33 (I7), U29.33 (I7)
- net pl6: now reaches U26.34 (I6)
- net pl6: now also U27.34 (I6), U28.34 (I6), U29.34 (I6)
- net pl5: now reaches U26.35 (I5)
- net pl5: now also U27.35 (I5), U28.35 (I5), U29.35 (I5)
- net at U26.37 (~{WE}): now also U27.37 (~{WE}), U28.37 (~{WE}), U29.37 (~{WE}), U29.40 (~{MSS/WRITE})
- net pl9: now reaches U26.38 (~{IEN})
- net pl9: now also U27.38 (~{IEN}), U28.38 (~{IEN}), U29.38 (~{IEN})
- net DA13: now reaches U26.4 (DA1)
- net DA13: now also U27.4 (DA1), U28.4 (DA1), U29.4 (DA1)
- net pl1: now reaches U26.41 (I1)
- net pl1: now also U27.41 (I1), U28.41 (I1), U29.41 (I1)
- net pl0: now reaches U26.42 (I0)
- net pl0: now also U27.42 (I0), U28.42 (I0), U29.42 (I0)
- net alu_b0: now reaches U26.44 (B0)
- net alu_b0: now also U27.44 (B0), U28.44 (B0), U29.44 (B0)
- net alu_b1: now reaches U26.45 (B1)
- net alu_b1: now also U27.45 (B1), U28.45 (B1), U29.45 (B1)
- net alu_b2: now reaches U26.46 (B2)
- net alu_b2: now also U27.46 (B2), U28.46 (B2), U29.46 (B2)
- net alu_b3: now reaches U26.47 (B3)
- net alu_b3: now also U27.47 (B3), U28.47 (B3), U29.47 (B3)
- net DA14: now reaches U26.5 (DA2)
- net DA14: now also U27.5 (DA2), U28.5 (DA2), U29.5 (DA2)
- net DA15: now reaches U26.6 (DA3)
- net DA15: now also U27.6 (DA3), U28.6 (DA3), U29.6 (DA3)
- net pl2: now reaches U26.7 (I2)
- net pl2: now also U27.7 (I2), U28.7 (I2), U29.7 (I2)
- net pl3: now reaches U26.8 (I3)
- net pl3: now also U27.8 (I3), U28.8 (I3), U29.8 (I3)
- net pl4: now reaches U26.9 (I4)
- net pl4: now also U27.9 (I4), U28.9 (I4), U29.9 (I4)
- net µ51: now reaches U25. (Vcc)
- net µ17: now reaches U33. (Vcc)
- net µ17: now also U35. (Vcc)
- new net: U28.12 (~{P}/OVR), U30.1 (~{G1})
- new net: U27.10 (CN), U30.11 (Cn+Y)
- new net: U28.10 (CN), U30.12 (Cn+X)
- new net: U29.10 (CN), U30.13 (Cn), U38.4 (Za)
- new net: U27.12 (~{P}/OVR), U30.14 (~{G2})
- new net: U27.14 (~{G}/N), U30.15 (~{P2})
- new net: U28.14 (~{G}/N), U30.2 (~{P1})
- new net: U29.12 (~{P}/OVR), U30.3 (~{G0})
- new net: U29.14 (~{G}/N), U30.4 (~{P0})
- new net: U28.20 (SIO0), U29.21 (SIO3)
- new net: U28.1 (QIO0), U29.48 (QIO3)
- new net: U27.1 (QIO0), U28.48 (QIO3)
- new net: U27.20 (SIO0), U28.21 (SIO3)
- new net: U33. (Vcc), U35. (Vcc), U36. (Vcc)
- new net: U33. (Vcc), U34. (Vcc), U35. (Vcc), U36. (Vcc) (x2)
- new net DB0: U21.2 (Y0)
- new net DB1: U21.5 (Y1)
- new net DB10: U20.6 (Y2)
- new net DB11: U20.9 (Y3)
- new net DB2: U21.6 (Y2)
- new net DB3: U21.9 (Y3)
- new net DB4: U21.12 (Y4)
- new net DB5: U21.15 (Y5)
- new net DB6: U21.16 (Y6)
- new net DB7: U21.19 (Y7)
- new net DB8: U20.2 (Y0)
- new net DB9: U20.5 (Y1)
- new net QL: U33. (Vcc), U34. (Vcc), U35. (Vcc)
- new net SL: U33. (Vcc), U34. (Vcc), U36. (Vcc)
- new net Y0: U29.16 (Y0)
- new net Y1: U29.17 (Y1)
- new net Y10: U27.18 (Y2)
- new net Y11: U27.19 (Y3)
- new net Y2: U29.18 (Y2)
- new net Y3: U29.19 (Y3)
- new net Y4: U28.16 (Y0)
- new net Y5: U28.17 (Y1)
- new net Y6: U28.18 (Y2)
- new net Y7: U28.19 (Y3)
- new net Y8: U27.16 (Y0)
- new net Y9: U27.17 (Y1)
- new net carry: U33. (Vcc), U34. (Vcc), U35. (Vcc), U36. (Vcc), U38.3 (I1a)
- new net pl: U38.1 (S)
- new net pl22: U20.21 (~{E}), U21.21 (~{E})
- new net pl35: U38.2 (I0a)
- new net ~{pl11}: U20.20 (~{OE}), U21.20 (~{OE})
- new net ~{pl8}: U35. (Vcc), U36. (Vcc)
- new net µ12: U34. (Vcc), U36. (Vcc)
- new net µ13: U34. (Vcc), U36. (Vcc)
- new net µ14: U34. (Vcc), U36. (Vcc)
- new net µ15: U33. (Vcc), U35. (Vcc)
- new net µ16: U33. (Vcc), U35. (Vcc)
- new net µ48: U25. (Vcc)
- new net µ49: U25. (Vcc)
- new net µ50: U25. (Vcc)
- no-connect marks 4 -> 27
Other:
- note added: "ERROR -> missing"
- moved on the sheet: U26, U33
